Commit message: Удалено лишнее.

File: src/UR5/ur5_single_arm_tufts/urdf/ur5_single_arm.urdf.xacro (robot description, xacro)
@@ -13,15 +13,4 @@
     <origin xyz="0 0 0" rpy="0 0 0"/>
   </xacro:robotiq_85_gripper>
-    <!-- kinect -->
-  <xacro:include filename="$(find ur5_single_arm_tufts)/urdf/sensors/kinect/kinect.urdf.xacro" />
-<!--   <xacro:kinect name="camera" parent="world" >
-    <origin xyz="0.6 0.0 1.8" rpy="0.0 ${pi/2} 0.0" />
-  </xacro:kinect> -->
-  <!-- kinect, ir, rgb sensor-->
-<!--   <xacro:include filename="$(find ur5_single_arm_tufts)/urdf/sensors/kinect2/common.xacro" />
-  <xacro:include filename="$(find ur5_single_arm_tufts)/urdf/sensors/kinect2/kinect2.urdf.xacro" />
-  <xacro:kinect2_v0 name="camera" parent="world" >
-    <origin xyz="0.4 0.0 1.2" rpy="0.0 ${pi/2} 0.0" />
-  </xacro:kinect2_v0> -->
   <!-- Pilar property -->
   <xacro:property name="pilar_height" value="0.09"/>

Commit message: Доработка сцены.

File: src/UR5/ur5_single_arm_tufts/urdf/ur5_single_arm.urdf.xacro (robot description, xacro)
@@ -14,5 +14,5 @@
   </xacro:robotiq_85_gripper>
   <!-- Pilar property -->
-  <xacro:property name="pilar_height" value="0.09"/>
+  <xacro:property name="pilar_height" value="0.2"/>
   <xacro:property name="pilar_radius" value="0.07"/>
   <link name="world"/>
