Commit message: Добавлена телега.

File: src/pkgs_ur5/ur5_single_arm_tufts/urdf/ur5_single_arm.urdf.xacro (robot description, xacro)
@@ -16,4 +16,6 @@
   <xacro:property name="pilar_height" value="0.2"/>
   <xacro:property name="pilar_radius" value="0.07"/>
+  <!-- <xacro:include filename="$(find husky_description)/urdf/husky.urdf.xacro" /> -->
+  <!-- <xacro:ur5_robot prefix="" joint_limited="false"/> -->
   <link name="world"/>
 <!--   <link name="table">
@@ -28,7 +30,7 @@
     <visual>
       <geometry>
-        <box size="1 1 0.05"/>
+        <box size="0.5 0.5 0.05"/>
       </geometry>
-      <material name="blue">
+      <material name="orange">
         <color rgba="0 0 .8 1"/>
       </material>
@@ -36,5 +38,5 @@
     <collision>
       <geometry>
-        <box size="1 1 0.05"/>
+        <box size="0.5 0.5 0.05"/>
       </geometry>
     </collision>
