Commit message: Добавлена рамка

File: src/ur5_husky_main/urdf/robot/husky.xacro (robot description, xacro)
@@ -22,4 +22,5 @@
     <xacro:include filename="$(find husky_description)/urdf/wheel.urdf.xacro" />
     <xacro:include filename="$(find husky_description)/urdf/accessories/intel_realsense.urdf.xacro"/>
+    <xacro:include filename="$(find husky_description)/urdf/accessories/sensor_arch.urdf.xacro"/>
     <xacro:property name="M_PI" value="3.14159"/>
     <!-- Base Size -->
@@ -34,4 +35,16 @@
     <xacro:property name="wheel_length" value="0.1143" />
     <xacro:property name="wheel_radius" value="0.1651" />
+    <!--
+      Add the main sensor arch if the user has specifically enabled it, or if a sensor
+      requires it for mounting
+    -->
+    <xacro:property name="sensorbar_user_enabled"     value="$(arg sensor_arch)" />
+    <xacro:property name="sensorbar_needed_realsense" value="$(arg realsense_enabled)" />
+    <xacro:property name="sensorbar_needed_lidar"     value="$(arg laser_3d_enabled)" />
+    <!-- <xacro:if value="${sensorbar_needed_realsense or sensorbar_user_enabled or sensorbar_needed_lidar}"> -->
+      <xacro:sensor_arch prefix="" parent="top_plate_link" size="$(arg sensor_arch_height)">
+          <origin xyz="$(optenv HUSKY_SENSOR_ARCH_OFFSET -0.32 0 0.51)" rpy="$(optenv HUSKY_SENSOR_ARCH_RPY 0 0 ${M_PI})"/>
+        </xacro:sensor_arch>
+    <!-- </xacro:if> -->
     <!-- Base link is the center of the robot's bottom plate -->
     <link name="base_link">

Commit message: Калибровка с реального робота.

File: src/ur5_husky_main/urdf/robot/husky.xacro (robot description, xacro)
@@ -19,6 +19,6 @@
     <xacro:arg name="cpr_urdf_extras" default="$(optenv CPR_URDF_EXTRAS empty.urdf)" />
     <!-- Included URDF/XACRO Files -->
-    <xacro:include filename="$(find husky_description)/urdf/decorations.urdf.xacro" />
-    <xacro:include filename="$(find husky_description)/urdf/wheel.urdf.xacro" />
+    <xacro:include filename="$(find ur5_husky_main)/urdf/robot/decorations.urdf.xacro" />
+    <xacro:include filename="$(find ur5_husky_main)/urdf/robot/wheel.urdf.xacro" />
     <xacro:include filename="$(find husky_description)/urdf/accessories/intel_realsense.urdf.xacro"/>
     <xacro:include filename="$(find husky_description)/urdf/accessories/sensor_arch.urdf.xacro"/>
@@ -34,5 +34,5 @@
     <!-- Wheel Properties -->
     <xacro:property name="wheel_length" value="0.1143" />
-    <xacro:property name="wheel_radius" value="0.1651" />
+    <xacro:property name="wheel_radius" value="0.1501" />
     <!--
       Add the main sensor arch if the user has specifically enabled it, or if a sensor

File: src/ur5_husky_main/urdf/robot/trajopt.xacro (robot description, xacro)
@@ -9,6 +9,6 @@
   <xacro:arg name="safety_k_position" default="20" /> <!-- Used to set k position in the safety controller-->
   <xacro:property name="prefix" value="ur5_"/>
-  <xacro:property name="wheel_radius" value="0.1651" />
-  <xacro:property name="wheel_vertical_offset" value="0.03282" />
+  <xacro:property name="wheel_radius" value="0.1501" />
+  <xacro:property name="wheel_vertical_offset" value="0.06" />
   <xacro:property name="M_PI" value="3.14159"/>
   <link name="world"/>
@@ -73,5 +73,6 @@
     <parent link="top_plate_link"/>
     <child link="${prefix}base_link"/>
-    <origin xyz="0.25 0.0 0.0" rpy="0 0 ${M_PI/2}"/>
+    <!--  Позиционирование робота на телеге -->
+    <origin xyz="0.3035 0.01 0.0" rpy="0 0 ${M_PI/2}"/>
   </joint>
 </robot>

File: src/ur5_husky_main/urdf/robot/ur5.xacro (robot description, xacro)
@@ -233,30 +233,9 @@
     </joint>
     <!-- Tool -->
-    <joint name="${prefix}add_length_tool_fixed" type="fixed">
+    <joint name="${prefix}ee_fixed_joint" type="fixed">
       <parent link="${prefix}wrist_3_link" />
-      <child link = "${prefix}add_length_tool" />
-      <origin xyz="0.0 0 0.03" rpy="0 0 0" />
-    </joint>
-    <link name="${prefix}add_length_tool">
-      <visual>
-        <origin rpy="0 0 0" xyz="0 0 0"/>
-        <geometry>
-          <cylinder length="0.06" radius="${wrist_3_inertia_radius}"/>
-        </geometry>
-        <material name="Black">
-          <color rgba="0 0 0 1"/>
-        </material>
-      </visual>
-      <collision>
-        <origin rpy="0 0 0" xyz="0 0 0"/>
-        <geometry>
-          <cylinder length="0.06" radius="${wrist_3_inertia_radius}"/>
-        </geometry>
-      </collision>
-    </link>
-    <joint name="${prefix}ee_fixed_joint" type="fixed">
-      <parent link="${prefix}add_length_tool" />
       <child link = "${prefix}ee_link" />
-      <origin xyz="0 0 0.035" rpy="0 ${pi/-2.0} 0" />
+      <!-- Корректировка offset гриппера -->
+      <origin xyz="0 0 0.015" rpy="0 ${pi/-2.0} 0" />
     </joint>
     <link name="${prefix}ee_link">
@@ -270,8 +249,9 @@
     <link name="${prefix}tool0"/>
     <joint name="${prefix}wrist_3_link-tool0_fixed_joint" type="fixed">
-      <origin xyz="0 0 0.06" rpy="0 0 0"/>
-      <parent link="${prefix}add_length_tool"/>
+      <origin xyz="0 0 0" rpy="${pi/-2.0} 0 0"/>
+      <parent link="${prefix}wrist_3_link"/>
       <child link="${prefix}tool0"/>
     </joint>
+    <!-- Floor base -->
     <xacro:ur_arm_transmission prefix="${prefix}" />
     <xacro:ur_arm_gazebo prefix="${prefix}" />
