Commit message: Доработка визуальной части. Цвет.

File: src/ur5_husky_main/urdf/robot/trajopt.xacro (robot description, xacro)
@@ -2,4 +2,7 @@
 <robot xmlns:xacro="http://ros.org/wiki/xacro" name="robot" >
   <xacro:property name="prefix" value="ur5_"/>
+  <xacro:property name="wheel_radius" value="0.1651" />
+  <xacro:property name="wheel_vertical_offset" value="0.03282" />
+  <xacro:property name="M_PI" value="3.14159"/>
   <link name="world"/>
   <!-- common stuff -->
@@ -21,5 +24,5 @@
     <parent link="world"/>
     <child link="base_link"/>
-    <origin xyz="0 0 0" rpy="0 0 0"/>
+    <origin xyz="0 0 ${wheel_radius - wheel_vertical_offset/2}" rpy="0 0 ${M_PI/2}"/>
   </joint>
   <joint name="ur5_to_base_link" type="fixed">

Commit message: Корректировка сцены.

File: src/ur5_husky_main/urdf/robot/trajopt.xacro (robot description, xacro)
@@ -24,5 +24,6 @@
     <parent link="world"/>
     <child link="base_link"/>
-    <origin xyz="0 0 ${wheel_radius - wheel_vertical_offset/2}" rpy="0 0 ${M_PI/2}"/>
+    <!-- не трогать xyz и rpy, иначе не считает траекторию! -->
+    <origin xyz="0 0 0" rpy="0 0 0"/>
   </joint>
   <joint name="ur5_to_base_link" type="fixed">

Commit message: Корректировка сцены.

File: src/ur5_husky_main/urdf/robot/trajopt.xacro (robot description, xacro)
@@ -6,4 +6,27 @@
   <xacro:property name="M_PI" value="3.14159"/>
   <link name="world"/>
+  <link name="floor">
+    <visual>
+        <origin xyz="0 0 -${wheel_radius - wheel_vertical_offset/2}" rpy="0 0 0" />
+        <geometry>
+          <box size="2 2 0.00005"/>
+        </geometry>
+        <material name="Floor">
+          <color rgba="0.72 0.80 0.97 0.7"/>
+        </material>
+      </visual>
+      <collision>
+        <origin xyz="0 0 -${wheel_radius - wheel_vertical_offset/2}" rpy="0 0 0" />
+        <geometry>
+          <box size="1 1 0.05"/>
+        </geometry>
+      </collision>
+      <collision>
+        <origin xyz="0 0 -${wheel_radius - wheel_vertical_offset/2}" rpy="0 0 0" />
+        <geometry>
+          <box size="1 1 0.05"/>
+        </geometry>
+      </collision>
+  </link>
   <!-- common stuff -->
   <xacro:include filename="$(find ur_description)/urdf/common.gazebo.xacro" />
@@ -21,6 +44,12 @@
   <xacro:include filename="$(find ur5_husky_main)/urdf/robot/husky.xacro" />
   <xacro:robot_husky />
-  <joint name="base_link_to_world" type="fixed">
+  <joint name="floor_to_world" type="fixed">
     <parent link="world"/>
+    <child link="floor"/>
+    <!-- не трогать xyz и rpy, иначе не считает траекторию! -->
+    <origin xyz="0 0 0" rpy="0 0 0"/>
+  </joint>
+  <joint name="base_link_to_floor" type="fixed">
+    <parent link="floor"/>
     <child link="base_link"/>
     <!-- не трогать xyz и rpy, иначе не считает траекторию! -->

Commit message: Правильное положение робота по отношению к тележке.

File: src/ur5_husky_main/urdf/robot/trajopt.xacro (robot description, xacro)
@@ -59,5 +59,5 @@
     <parent link="top_plate_link"/>
     <child link="${prefix}base_link"/>
-    <origin xyz="0.25 0.0 0.0" rpy="0 0 0"/>
+    <origin xyz="0.25 0.0 0.0" rpy="0 0 -${M_PI/2}"/>
   </joint>
 </robot>

Commit message: Движение через несколько положений. Плавное движение.

File: src/ur5_husky_main/urdf/robot/trajopt.xacro (robot description, xacro)
@@ -60,4 +60,6 @@
     <child link="${prefix}base_link"/>
     <origin xyz="0.25 0.0 0.0" rpy="0 0 -${M_PI/2}"/>
+    <!-- не трогать xyz и rpy, иначе не считает траекторию! -->
+    <!-- <origin xyz="0.25 0.0 0.0" rpy="0 0 0"/> -->
   </joint>
 </robot>

Commit message: Попытка калибровки робота

File: src/ur5_husky_main/urdf/robot/trajopt.xacro (robot description, xacro)
@@ -1,4 +1,5 @@
 <?xml version="1.0"?>
 <robot xmlns:xacro="http://ros.org/wiki/xacro" name="robot" >
+  <xacro:arg name="kinematics_parameters_file" default="$(find ur5_husky_main)/config/robot_calibration.yaml"/>
   <xacro:property name="prefix" value="ur5_"/>
   <xacro:property name="wheel_radius" value="0.1651" />
@@ -32,7 +33,7 @@
   <xacro:include filename="$(find ur_description)/urdf/common.gazebo.xacro" />
   <!-- ur5 -->
-  <xacro:include filename="$(find ur_description)/urdf/ur5.urdf.xacro" />
+  <xacro:include filename="$(find ur5_husky_main)/urdf/robot/ur5.xacro" />
   <!-- arm -->
-  <xacro:ur5_robot prefix="${prefix}" joint_limited="false"/>
+  <xacro:ur5_robot prefix="${prefix}" joint_limited="false" kinematics_parameters_file="$(arg kinematics_parameters_file)"/>
   <!-- robotiq 85 -->
   <xacro:include filename="$(find robotiq_85_description)/urdf/robotiq_85_gripper.urdf.xacro" />

File: src/ur5_husky_main/urdf/robot/ur5.xacro (robot description, xacro)
@@ -3,5 +3,14 @@
   <xacro:include filename="$(find ur_description)/urdf/ur.transmission.xacro" />
   <xacro:include filename="$(find ur_description)/urdf/ur.gazebo.xacro" />
-  <xacro:macro name="ur5_robot" params="prefix joint_limited
+  <xacro:macro name="cylinder_inertial" params="radius length mass *origin">
+    <inertial>
+      <mass value="${mass}" />
+      <xacro:insert_block name="origin" />
+      <inertia ixx="${0.0833333 * mass * (3 * radius * radius + length * length)}" ixy="0.0" ixz="0.0"
+        iyy="${0.0833333 * mass * (3 * radius * radius + length * length)}" iyz="0.0"
+        izz="${0.5 * mass * radius * radius}" />
+    </inertial>
+  </xacro:macro>
+  <xacro:macro name="ur5_robot" params="prefix joint_limited kinematics_parameters_file
      shoulder_pan_lower_limit:=${-pi}    shoulder_pan_upper_limit:=${pi}
      shoulder_lift_lower_limit:=${-pi}    shoulder_lift_upper_limit:=${pi}
@@ -10,4 +19,7 @@
      wrist_2_lower_limit:=${-pi}    wrist_2_upper_limit:=${pi}
      wrist_3_lower_limit:=${-pi}    wrist_3_upper_limit:=${pi}">
+    <!-- Load calibration params -->
+    <xacro:property name="config_kinematics_parameters" value="${load_yaml(kinematics_parameters_file)}"/>
+    <xacro:property name="sec_kinematics" value="${config_kinematics_parameters['kinematics']}" />
     <!-- Inertia parameters -->
     <xacro:property name="base_mass" value="4.0" />  <!-- This mass might be incorrect -->
@@ -24,4 +36,16 @@
     <xacro:property name="wrist_2_cog" value="0.0 0.0018 0.11099" />
     <xacro:property name="wrist_3_cog" value="0.0 0.001159 0.0" />
+    <!-- Kinematic model -->
+    <!-- Properties from urcontrol.conf -->
+    <!--
+      DH for UR5:
+      a = [0.00000, -0.42500, -0.39225,  0.00000,  0.00000,  0.0000]
+      d = [0.089159,  0.00000,  0.00000,  0.10915,  0.09465,  0.0823]
+      alpha = [ 1.570796327, 0, 0, 1.570796327, -1.570796327, 0 ]
+      q_home_offset = [0, -1.570796327, 0, -1.570796327, 0, 0]
+      joint_direction = [-1, -1, 1, 1, 1, 1]
+      mass = [3.7000, 8.3930, 2.2750, 1.2190, 1.2190, 0.1879]
+      center_of_mass = [ [0, -0.02561, 0.00193], [0.2125, 0, 0.11336], [0.11993, 0.0, 0.0265], [0, -0.0018, 0.01634], [0, 0.0018,0.01634], [0, 0, -0.001159] ]
+    -->
     <xacro:property name="d1" value="0.089159" />
     <xacro:property name="a2" value="-0.42500" />
@@ -30,4 +54,47 @@
     <xacro:property name="d5" value="0.09465" />
     <xacro:property name="d6" value="0.0823" />
+    <!-- kinematics -->
+    <xacro:property name="shoulder_x" value="${sec_kinematics['shoulder']['x']}" scope="parent"/>
+    <xacro:property name="shoulder_y" value="${sec_kinematics['shoulder']['y']}" scope="parent"/>
+    <xacro:property name="shoulder_z" value="${sec_kinematics['shoulder']['z']}" scope="parent"/>
+    <xacro:property name="shoulder_roll" value="${sec_kinematics['shoulder']['roll']}" scope="parent"/>
+    <xacro:property name="shoulder_pitch" value="${sec_kinematics['shoulder']['pitch']}" scope="parent"/>
+    <xacro:property name="shoulder_yaw" value="${sec_kinematics['shoulder']['yaw']}" scope="parent"/>
+    <xacro:property name="upper_arm_x" value="${sec_kinematics['upper_arm']['x']}" scope="parent"/>
+    <xacro:property name="upper_arm_y" value="${sec_kinematics['upper_arm']['y']}" scope="parent"/>
+    <xacro:property name="upper_arm_z" value="${sec_kinematics['upper_arm']['z']}" scope="parent"/>
+    <xacro:property name="upper_arm_roll" value="${sec_kinematics['upper_arm']['roll']}" scope="parent"/>
+    <xacro:property name="upper_arm_pitch" value="${sec_kinematics['upper_arm']['pitch']}" scope="parent"/>
+    <xacro:property name="upper_arm_yaw" value="${sec_kinematics['upper_arm']['yaw']}" scope="parent"/>
+    <xacro:property name="forearm_x" value="${sec_kinematics['forearm']['x']}" scope="parent"/>
+    <xacro:property name="forearm_y" value="${sec_kinematics['forearm']['y']}" scope="parent"/>
+    <xacro:property name="forearm_z" value="${sec_kinematics['forearm']['z']}" scope="parent"/>
+    <xacro:property name="forearm_roll" value="${sec_kinematics['forearm']['roll']}" scope="parent"/>
+    <xacro:property name="forearm_pitch" value="${sec_kinematics['forearm']['pitch']}" scope="parent"/>
+    <xacro:property name="forearm_yaw" value="${sec_kinematics['forearm']['yaw']}" scope="parent"/>
+    <xacro:property name="wrist_1_x" value="${sec_kinematics['wrist_1']['x']}" scope="parent"/>
+    <xacro:property name="wrist_1_y" value="${sec_kinematics['wrist_1']['y']}" scope="parent"/>
+    <xacro:property name="wrist_1_z" value="${sec_kinematics['wrist_1']['z']}" scope="parent"/>
+    <xacro:property name="wrist_1_roll" value="${sec_kinematics['wrist_1']['roll']}" scope="parent"/>
+    <xacro:property name="wrist_1_pitch" value="${sec_kinematics['wrist_1']['pitch']}" scope="parent"/>
+    <xacro:property name="wrist_1_yaw" value="${sec_kinematics['wrist_1']['yaw']}" scope="parent"/>
+    <xacro:property name="wrist_2_x" value="${sec_kinematics['wrist_2']['x']}" scope="parent"/>
+    <xacro:property name="wrist_2_y" value="${sec_kinematics['wrist_2']['y']}" scope="parent"/>
+    <xacro:property name="wrist_2_z" value="${sec_kinematics['wrist_2']['z']}" scope="parent"/>
+    <xacro:property name="wrist_2_roll" value="${sec_kinematics['wrist_2']['roll']}" scope="parent"/>
+    <xacro:property name="wrist_2_pitch" value="${sec_kinematics['wrist_2']['pitch']}" scope="parent"/>
+    <xacro:property name="wrist_2_yaw" value="${sec_kinematics['wrist_2']['yaw']}" scope="parent"/>
+    <xacro:property name="wrist_3_x" value="${sec_kinematics['wrist_3']['x']}" scope="parent"/>
+    <xacro:property name="wrist_3_y" value="${sec_kinematics['wrist_3']['y']}" scope="parent"/>
+    <xacro:property name="wrist_3_z" value="${sec_kinematics['wrist_3']['z']}" scope="parent"/>
+    <xacro:property name="wrist_3_roll" value="${sec_kinematics['wrist_3']['roll']}" scope="parent"/>
+    <xacro:property name="wrist_3_pitch" value="${sec_kinematics['wrist_3']['pitch']}" scope="parent"/>
+    <xacro:property name="wrist_3_yaw" value="${sec_kinematics['wrist_3']['yaw']}" scope="parent"/>
+<!--     <xacro:property name="d1" value="0.08956401716053501" />
+    <xacro:property name="a2" value="-0.4252719934925572" />
+    <xacro:property name="a3" value="-0.3920768556643368" />
+    <xacro:property name="d4" value="0.1103173677297831" />
+    <xacro:property name="d5" value="0.09477508287480087" />
+    <xacro:property name="d6" value="0.08249382179030061" /> -->
     <!-- Arbitrary offsets for shoulder/elbow joints -->
     <xacro:property name="shoulder_offset" value="0.13585" />  <!-- measured from model -->
@@ -66,5 +133,5 @@
       <parent link="${prefix}base_link" />
       <child link = "${prefix}shoulder_link" />
-      <origin xyz="0.0 0.0 ${shoulder_height}" rpy="0.0 0.0 0.0" />
+      <origin xyz="${shoulder_x} ${shoulder_y} ${shoulder_z}" rpy="${shoulder_roll} ${shoulder_pitch} ${shoulder_yaw}" />
       <axis xyz="0 0 1" />
       <xacro:unless value="${joint_limited}">
@@ -97,5 +164,5 @@
       <parent link="${prefix}shoulder_link" />
       <child link = "${prefix}upper_arm_link" />
-      <origin xyz="0.0 ${shoulder_offset} 0.0" rpy="0.0 ${pi / 2.0} 0.0" />
+      <origin xyz="${upper_arm_x} ${upper_arm_y} ${upper_arm_z}" rpy="${upper_arm_roll} ${upper_arm_pitch} ${upper_arm_yaw}" />
       <axis xyz="0 1 0" />
       <xacro:unless value="${joint_limited}">
@@ -128,5 +195,5 @@
       <parent link="${prefix}upper_arm_link" />
       <child link = "${prefix}forearm_link" />
-      <origin xyz="0.0 ${elbow_offset} ${upper_arm_length}" rpy="0.0 0.0 0.0" />
+      <origin xyz="${forearm_x} ${forearm_y} ${forearm_z}" rpy="${forearm_roll} ${forearm_pitch} ${forearm_yaw}" />
       <axis xyz="0 1 0" />
       <xacro:unless value="${joint_limited}">
@@ -159,5 +226,5 @@
       <parent link="${prefix}forearm_link" />
       <child link = "${prefix}wrist_1_link" />
-      <origin xyz="0.0 0.0 ${forearm_length}" rpy="0.0 ${pi / 2.0} 0.0" />
+      <origin xyz="${wrist_1_x} ${wrist_1_y} ${wrist_1_z}" rpy="${wrist_1_roll} ${wrist_1_pitch} ${wrist_1_yaw}" />
       <axis xyz="0 1 0" />
       <xacro:unless value="${joint_limited}">
@@ -190,5 +257,5 @@
       <parent link="${prefix}wrist_1_link" />
       <child link = "${prefix}wrist_2_link" />
-      <origin xyz="0.0 ${wrist_1_length} 0.0" rpy="0.0 0.0 0.0" />
+      <origin xyz="${wrist_2_x} ${wrist_2_y} ${wrist_2_z}" rpy="${wrist_2_roll} ${wrist_2_pitch} ${wrist_2_yaw}" />
       <axis xyz="0 0 1" />
       <xacro:unless value="${joint_limited}">
@@ -221,5 +288,5 @@
       <parent link="${prefix}wrist_2_link" />
       <child link = "${prefix}wrist_3_link" />
-      <origin xyz="0.0 0.0 ${wrist_2_length}" rpy="0.0 0.0 0.0" />
+      <origin xyz="${wrist_3_x} ${wrist_3_y} ${wrist_3_z}" rpy="${wrist_3_roll} ${wrist_3_pitch} ${wrist_3_yaw}" />
       <axis xyz="0 1 0" />
       <xacro:unless value="${joint_limited}">
