Commit message: Калибровка робота.

File: src/ur5_husky_main/urdf/robot/trajopt.xacro (robot description, xacro)
@@ -1,5 +1,11 @@
 <?xml version="1.0"?>
 <robot xmlns:xacro="http://ros.org/wiki/xacro" name="robot" >
-  <xacro:arg name="kinematics_parameters_file" default="$(find ur5_husky_main)/config/robot_calibration.yaml"/>
+  <xacro:arg name="kinematics_parameters_file" default="$(find ur5_husky_main)/config/ur5/default_kinematics.yaml"/>
+  <xacro:arg name="physical_parameters_file" default="$(find ur5_husky_main)/config/ur5/physical_parameters.yaml"/>
+  <xacro:arg name="joint_limits_parameters_file" default="$(find ur5_husky_main)/config/ur5/joint_limits.yaml"/>
+  <xacro:arg name="visual_parameters_file" default="$(find ur5_husky_main)/config/ur5/visual_parameters_file.yaml"/>
+  <xacro:arg name="safety_limits" default="false" /> <!-- If True, enable the safety limits controller -->
+  <xacro:arg name="safety_pos_margin" default="0.15" /> <!-- The lower/upper limits in the safety controller -->
+  <xacro:arg name="safety_k_position" default="20" /> <!-- Used to set k position in the safety controller-->
   <xacro:property name="prefix" value="ur5_"/>
   <xacro:property name="wheel_radius" value="0.1651" />
@@ -35,10 +41,17 @@
   <xacro:include filename="$(find ur5_husky_main)/urdf/robot/ur5.xacro" />
   <!-- arm -->
-  <xacro:ur5_robot prefix="${prefix}" joint_limited="false" kinematics_parameters_file="$(arg kinematics_parameters_file)"/>
+  <xacro:ur5_robot prefix="${prefix}"
+    kinematics_parameters_file="$(arg kinematics_parameters_file)"
+    physical_parameters_file="$(arg physical_parameters_file)"
+    joint_limits_parameters_file="$(arg joint_limits_parameters_file)"
+    visual_parameters_file="$(arg visual_parameters_file)"
+    safety_limits="$(arg safety_limits)"
+    safety_pos_margin="$(arg safety_pos_margin)"
+    safety_k_position="$(arg safety_k_position)"/>
   <!-- robotiq 85 -->
   <xacro:include filename="$(find robotiq_85_description)/urdf/robotiq_85_gripper.urdf.xacro" />
   <!-- gripper -->
   <xacro:robotiq_85_gripper prefix="" parent="${prefix}ee_link" >
-    <origin xyz="0 0 0" rpy="0 0 0"/>
+    <origin xyz="0 0 0" rpy="${M_PI/2} 0 0"/>
   </xacro:robotiq_85_gripper>
   <!-- husky -->
@@ -60,7 +73,5 @@
     <parent link="top_plate_link"/>
     <child link="${prefix}base_link"/>
-    <origin xyz="0.25 0.0 0.0" rpy="0 0 -${M_PI/2}"/>
-    <!-- не трогать xyz и rpy, иначе не считает траекторию! -->
-    <!-- <origin xyz="0.25 0.0 0.0" rpy="0 0 0"/> -->
+    <origin xyz="0.25 0.0 0.0" rpy="0 0 ${M_PI/2}"/>
   </joint>
 </robot>

File: src/ur5_husky_main/urdf/robot/ur5.xacro (robot description, xacro)
@@ -3,5 +3,6 @@
   <xacro:include filename="$(find ur_description)/urdf/ur.transmission.xacro" />
   <xacro:include filename="$(find ur_description)/urdf/ur.gazebo.xacro" />
-  <xacro:macro name="cylinder_inertial" params="radius length mass *origin">
+  <xacro:include filename="$(find ur5_husky_main)/urdf/robot/ur5_common.xacro" />
+<!--   <xacro:macro name="cylinder_inertial" params="radius length mass *origin">
     <inertial>
       <mass value="${mass}" />
@@ -11,18 +12,27 @@
         izz="${0.5 * mass * radius * radius}" />
     </inertial>
-  </xacro:macro>
-  <xacro:macro name="ur5_robot" params="prefix joint_limited kinematics_parameters_file
-     shoulder_pan_lower_limit:=${-pi}    shoulder_pan_upper_limit:=${pi}
-     shoulder_lift_lower_limit:=${-pi}    shoulder_lift_upper_limit:=${pi}
-     elbow_joint_lower_limit:=${-pi}    elbow_joint_upper_limit:=${pi}
-     wrist_1_lower_limit:=${-pi}    wrist_1_upper_limit:=${pi}
-     wrist_2_lower_limit:=${-pi}    wrist_2_upper_limit:=${pi}
-     wrist_3_lower_limit:=${-pi}    wrist_3_upper_limit:=${pi}">
+  </xacro:macro> -->
+  <xacro:macro name="ur5_robot" params="
+    prefix
+    joint_limits_parameters_file
+    kinematics_parameters_file
+    physical_parameters_file
+    visual_parameters_file
+    safety_limits:=false
+    safety_pos_margin:=0.15
+    safety_k_position:=20
+    ">
+    <!-- Load configuration data from the provided .yaml files -->
+    <xacro:read_model_data
+      joint_limits_parameters_file="${joint_limits_parameters_file}"
+      kinematics_parameters_file="${kinematics_parameters_file}"
+      physical_parameters_file="${physical_parameters_file}"
+      visual_parameters_file="${visual_parameters_file}"/>
     <!-- Load calibration params -->
-    <xacro:property name="config_kinematics_parameters" value="${load_yaml(kinematics_parameters_file)}"/>
-    <xacro:property name="sec_kinematics" value="${config_kinematics_parameters['kinematics']}" />
+<!--     <xacro:property name="config_kinematics_parameters" value="${load_yaml(kinematics_parameters_file)}"/>
+    <xacro:property name="sec_kinematics" value="${config_kinematics_parameters['kinematics']}" /> -->
     <!-- Inertia parameters -->
-    <xacro:property name="base_mass" value="4.0" />  <!-- This mass might be incorrect -->
-    <xacro:property name="shoulder_mass" value="3.7000" />
+<!--     <xacro:property name="base_mass" value="4.0" />  --> <!-- This mass might be incorrect -->
+<!--     <xacro:property name="shoulder_mass" value="3.7000" />
     <xacro:property name="upper_arm_mass" value="8.3930" />
     <xacro:property name="forearm_mass" value="2.2750" />
@@ -35,5 +45,5 @@
     <xacro:property name="wrist_1_cog" value="0.0 0.110949 0.01634" />
     <xacro:property name="wrist_2_cog" value="0.0 0.0018 0.11099" />
-    <xacro:property name="wrist_3_cog" value="0.0 0.001159 0.0" />
+    <xacro:property name="wrist_3_cog" value="0.0 0.001159 0.0" /> -->
     <!-- Kinematic model -->
     <!-- Properties from urcontrol.conf -->
@@ -48,12 +58,12 @@
       center_of_mass = [ [0, -0.02561, 0.00193], [0.2125, 0, 0.11336], [0.11993, 0.0, 0.0265], [0, -0.0018, 0.01634], [0, 0.0018,0.01634], [0, 0, -0.001159] ]
     -->
-    <xacro:property name="d1" value="0.089159" />
+   <!--  <xacro:property name="d1" value="0.089159" />
     <xacro:property name="a2" value="-0.42500" />
     <xacro:property name="a3" value="-0.39225" />
     <xacro:property name="d4" value="0.10915" />
     <xacro:property name="d5" value="0.09465" />
-    <xacro:property name="d6" value="0.0823" />
+    <xacro:property name="d6" value="0.0823" /> -->
     <!-- kinematics -->
-    <xacro:property name="shoulder_x" value="${sec_kinematics['shoulder']['x']}" scope="parent"/>
+<!--     <xacro:property name="shoulder_x" value="${sec_kinematics['shoulder']['x']}" scope="parent"/>
     <xacro:property name="shoulder_y" value="${sec_kinematics['shoulder']['y']}" scope="parent"/>
     <xacro:property name="shoulder_z" value="${sec_kinematics['shoulder']['z']}" scope="parent"/>
@@ -90,16 +100,13 @@
     <xacro:property name="wrist_3_roll" value="${sec_kinematics['wrist_3']['roll']}" scope="parent"/>
     <xacro:property name="wrist_3_pitch" value="${sec_kinematics['wrist_3']['pitch']}" scope="parent"/>
-    <xacro:property name="wrist_3_yaw" value="${sec_kinematics['wrist_3']['yaw']}" scope="parent"/>
-<!--     <xacro:property name="d1" value="0.08956401716053501" />
-    <xacro:property name="a2" value="-0.4252719934925572" />
-    <xacro:property name="a3" value="-0.3920768556643368" />
-    <xacro:property name="d4" value="0.1103173677297831" />
-    <xacro:property name="d5" value="0.09477508287480087" />
-    <xacro:property name="d6" value="0.08249382179030061" /> -->
+    <xacro:property name="wrist_3_yaw" value="${sec_kinematics['wrist_3']['yaw']}" scope="parent"/> -->
     <!-- Arbitrary offsets for shoulder/elbow joints -->
-    <xacro:property name="shoulder_offset" value="0.13585" />  <!-- measured from model -->
-    <xacro:property name="elbow_offset" value="-0.1197" /> <!-- measured from model -->
+<!--     <xacro:property name="shoulder_offset" value="0.13585" />
+    <xacro:property name="elbow_offset" value="-0.1197" />
+    <xacro:property name="wrist_1_visual_offset" value="-0.093" scope="parent"/>
+    <xacro:property name="wrist_2_visual_offset" value="-0.095" scope="parent"/>
+    <xacro:property name="wrist_3_visual_offset" value="-0.0818" scope="parent"/> -->
     <!-- link lengths used in model -->
-    <xacro:property name="shoulder_height" value="${d1}" />
+<!--     <xacro:property name="shoulder_height" value="${d1}" />
     <xacro:property name="upper_arm_length" value="${-a2}" />
     <xacro:property name="forearm_length" value="${-a3}" />
@@ -107,10 +114,10 @@
     <xacro:property name="wrist_2_length" value="${d5}" />
     <xacro:property name="wrist_3_length" value="${d6}" />
-    <xacro:property name="shoulder_radius" value="0.060" />   <!-- manually measured -->
-    <xacro:property name="upper_arm_radius" value="0.054" />  <!-- manually measured -->
-    <xacro:property name="elbow_radius" value="0.060" />      <!-- manually measured -->
-    <xacro:property name="forearm_radius" value="0.040" />    <!-- manually measured -->
-    <xacro:property name="wrist_radius" value="0.045" />      <!-- manually measured -->
-    <link name="${prefix}base_link" >
+    <xacro:property name="shoulder_radius" value="0.060" />
+    <xacro:property name="upper_arm_radius" value="0.054" />
+    <xacro:property name="elbow_radius" value="0.060" />
+    <xacro:property name="forearm_radius" value="0.040" />
+    <xacro:property name="wrist_radius" value="0.045" />  -->
+<!--      <link name="${prefix}base_link" >
       <visual>
         <geometry>
@@ -129,195 +136,244 @@
         <origin xyz="0.0 0.0 0.0" rpy="0 0 0" />
       </xacro:cylinder_inertial>
+    </link> -->
+    <link name="${prefix}base_link">
+      <visual>
+        <origin xyz="0 0 0" rpy="0 0 ${pi}"/>
+        <geometry>
+          <mesh filename="${base_visual_mesh}"/>
+        </geometry>
+        <material name="${base_visual_material_name}">
+          <color rgba="${base_visual_material_color}"/>
+        </material>
+      </visual>
+      <collision>
+        <origin xyz="0 0 0" rpy="0 0 ${pi}"/>
+        <geometry>
+          <mesh filename="${base_collision_mesh}"/>
+        </geometry>
+      </collision>
+      <xacro:cylinder_inertial radius="${base_inertia_radius}" length="${base_inertia_length}" mass="${base_mass}">
+        <origin xyz="0 0 0" rpy="0 0 0" />
+      </xacro:cylinder_inertial>
+    </link>
+    <link name="${prefix}shoulder_link">
+      <visual>
+        <origin xyz="0 0 0" rpy="0 0 ${pi}"/>
+        <geometry>
+          <mesh filename="${shoulder_visual_mesh}"/>
+        </geometry>
+        <material name="${shoulder_visual_material_name}">
+          <color rgba="${shoulder_visual_material_color}"/>
+        </material>
+      </visual>
+      <collision>
+        <origin xyz="0 0 0" rpy="0 0 ${pi}"/>
+        <geometry>
+          <mesh filename="${shoulder_collision_mesh}"/>
+        </geometry>
+      </collision>
+      <xacro:cylinder_inertial radius="${shoulder_inertia_radius}" length="${shoulder_inertia_length}" mass="${shoulder_mass}">
+        <origin xyz="0 0 0" rpy="0 0 0" />
+      </xacro:cylinder_inertial>
+    </link>
+    <link name="${prefix}upper_arm_link">
+      <visual>
+        <origin xyz="0 0 ${shoulder_offset}" rpy="${pi/2} 0 ${-pi/2}"/>
+        <geometry>
+          <mesh filename="${upper_arm_visual_mesh}"/>
+        </geometry>
+        <material name="${upper_arm_visual_material_name}">
+          <color rgba="${upper_arm_visual_material_color}"/>
+        </material>
+      </visual>
+      <collision>
+        <origin xyz="0 0 ${shoulder_offset}" rpy="${pi/2} 0 ${-pi/2}"/>
+        <geometry>
+          <mesh filename="${upper_arm_collision_mesh}"/>
+        </geometry>
+      </collision>
+      <xacro:cylinder_inertial radius="${upperarm_inertia_radius}" length="${upperarm_inertia_length}" mass="${upper_arm_mass}">
+        <origin xyz="${-0.5 * upperarm_inertia_length} 0.0 ${upper_arm_inertia_offset}" rpy="0 ${pi/2} 0" />
+      </xacro:cylinder_inertial>
+    </link>
+    <link name="${prefix}forearm_link">
+      <visual>
+        <origin xyz="0 0 ${elbow_offset}" rpy="${pi/2} 0 ${-pi/2}"/>
+        <geometry>
+          <mesh filename="${forearm_visual_mesh}"/>
+        </geometry>
+        <material name="${forearm_visual_material_name}">
+          <color rgba="${forearm_visual_material_color}"/>
+        </material>
+      </visual>
+      <collision>
+        <origin xyz="0 0 ${elbow_offset}" rpy="${pi/2} 0 ${-pi/2}"/>
+        <geometry>
+          <mesh filename="${forearm_collision_mesh}"/>
+        </geometry>
+      </collision>
+      <xacro:cylinder_inertial radius="${forearm_inertia_radius}" length="${forearm_inertia_length}"  mass="${forearm_mass}">
+        <origin xyz="${-0.5 * forearm_inertia_length} 0.0 ${elbow_offset}" rpy="0 ${pi/2} 0" />
+      </xacro:cylinder_inertial>
+    </link>
+    <link name="${prefix}wrist_1_link">
+      <visual>
+       <origin xyz="0 0 ${wrist_1_visual_offset}" rpy="${pi/2} 0 0"/>
+        <geometry>
+          <mesh filename="${wrist_1_visual_mesh}"/>
+        </geometry>
+        <material name="${wrist_1_visual_material_name}">
+          <color rgba="${wrist_1_visual_material_color}"/>
+        </material>
+      </visual>
+      <collision>
+        <origin xyz="0 0 ${wrist_1_visual_offset}" rpy="${pi/2} 0 0"/>
+        <geometry>
+          <mesh filename="${wrist_1_collision_mesh}"/>
+        </geometry>
+      </collision>
+      <xacro:cylinder_inertial radius="${wrist_1_inertia_radius}" length="${wrist_1_inertia_length}"  mass="${wrist_1_mass}">
+        <origin xyz="0 0 0" rpy="0 0 0" />
+      </xacro:cylinder_inertial>
+    </link>
+    <link name="${prefix}wrist_2_link">
+      <visual>
+        <origin xyz="0 0 ${wrist_2_visual_offset}" rpy="0 0 0"/>
+        <geometry>
+          <mesh filename="${wrist_2_visual_mesh}"/>
+        </geometry>
+        <material name="${wrist_2_visual_material_name}">
+          <color rgba="${wrist_2_visual_material_color}"/>
+        </material>
+      </visual>
+      <collision>
+        <origin xyz="0 0 ${wrist_2_visual_offset}" rpy="0 0 0"/>
+        <geometry>
+          <mesh filename="${wrist_2_collision_mesh}"/>
+        </geometry>
+      </collision>
+      <xacro:cylinder_inertial radius="${wrist_2_inertia_radius}" length="${wrist_2_inertia_length}"  mass="${wrist_2_mass}">
+        <origin xyz="0 0 0" rpy="0 0 0" />
+      </xacro:cylinder_inertial>
+    </link>
+    <link name="${prefix}wrist_3_link">
+      <visual>
+        <origin xyz="0 0 ${wrist_3_visual_offset}" rpy="${pi/2} 0 0"/>
+        <geometry>
+          <mesh filename="${wrist_3_visual_mesh}"/>
+        </geometry>
+        <material name="${wrist_3_visual_material_name}">
+          <color rgba="${wrist_3_visual_material_color}"/>
+        </material>
+      </visual>
+      <collision>
+        <origin xyz="0 0 ${wrist_3_visual_offset}" rpy="${pi/2} 0 0"/>
+        <geometry>
+          <mesh filename="${wrist_3_collision_mesh}"/>
+        </geometry>
+      </collision>
+      <xacro:cylinder_inertial radius="${wrist_3_inertia_radius}" length="${wrist_3_inertia_length}"  mass="${wrist_3_mass}">
+        <origin xyz="0.0 0.0 ${-0.5 * wrist_3_inertia_length}" rpy="0 0 0" />
+      </xacro:cylinder_inertial>
     </link>
     <joint name="${prefix}shoulder_pan_joint" type="revolute">
       <parent link="${prefix}base_link" />
-      <child link = "${prefix}shoulder_link" />
+      <child link="${prefix}shoulder_link" />
       <origin xyz="${shoulder_x} ${shoulder_y} ${shoulder_z}" rpy="${shoulder_roll} ${shoulder_pitch} ${shoulder_yaw}" />
       <axis xyz="0 0 1" />
-      <xacro:unless value="${joint_limited}">
-        <limit lower="${-2.0 * pi}" upper="${2.0 * pi}" effort="150.0" velocity="3.15"/>
-      </xacro:unless>
-      <xacro:if value="${joint_limited}">
-        <limit lower="${shoulder_pan_lower_limit}" upper="${shoulder_pan_upper_limit}" effort="150.0" velocity="3.15"/>
-      </xacro:if>
-      <dynamics damping="0.0" friction="0.0"/>
-    </joint>
-    <link name="${prefix}shoulder_link">
-      <visual>
-        <geometry>
-          <mesh filename="package://ur_description/meshes/ur5/visual/shoulder.dae" />
-        </geometry>
-        <material name="LightGrey">
-          <color rgba="0.7 0.7 0.7 1.0"/>
-        </material>
-      </visual>
-      <collision>
-        <geometry>
-          <mesh filename="package://ur_description/meshes/ur5/collision/shoulder.stl" />
-        </geometry>
-      </collision>
-      <xacro:cylinder_inertial radius="0.06" length="0.15" mass="${shoulder_mass}">
-        <origin xyz="0.0 0.0 0.0" rpy="0 0 0" />
-      </xacro:cylinder_inertial>
-    </link>
+      <limit lower="${shoulder_pan_lower_limit}" upper="${shoulder_pan_upper_limit}"
+        effort="${shoulder_pan_effort_limit}" velocity="${shoulder_pan_velocity_limit}"/>
+      <xacro:if value="${safety_limits}">
+         <safety_controller soft_lower_limit="${shoulder_pan_lower_limit + safety_pos_margin}" soft_upper_limit="${shoulder_pan_upper_limit - safety_pos_margin}" k_position="${safety_k_position}" k_velocity="0.0"/>
+      </xacro:if>
+      <dynamics damping="0" friction="0"/>
+    </joint>
     <joint name="${prefix}shoulder_lift_joint" type="revolute">
       <parent link="${prefix}shoulder_link" />
-      <child link = "${prefix}upper_arm_link" />
+      <child link="${prefix}upper_arm_link" />
       <origin xyz="${upper_arm_x} ${upper_arm_y} ${upper_arm_z}" rpy="${upper_arm_roll} ${upper_arm_pitch} ${upper_arm_yaw}" />
-      <axis xyz="0 1 0" />
-      <xacro:unless value="${joint_limited}">
-        <limit lower="${-2.0 * pi}" upper="${2.0 * pi}" effort="150.0" velocity="3.15"/>
-      </xacro:unless>
-      <xacro:if value="${joint_limited}">
-        <limit lower="${shoulder_lift_lower_limit}" upper="${shoulder_lift_upper_limit}" effort="150.0" velocity="3.15"/>
-      </xacro:if>
-      <dynamics damping="0.0" friction="0.0"/>
-    </joint>
-    <link name="${prefix}upper_arm_link">
-      <visual>
-        <geometry>
-          <mesh filename="package://ur_description/meshes/ur5/visual/upperarm.dae" />
-        </geometry>
-        <material name="LightGrey">
-          <color rgba="0.7 0.7 0.7 1.0"/>
-        </material>
-      </visual>
-      <collision>
-        <geometry>
-          <mesh filename="package://ur_description/meshes/ur5/collision/upperarm.stl" />
-        </geometry>
-      </collision>
-      <xacro:cylinder_inertial radius="0.06" length="0.56" mass="${upper_arm_mass}">
-        <origin xyz="0.0 0.0 0.28" rpy="0 0 0" />
-      </xacro:cylinder_inertial>
-    </link>
+      <axis xyz="0 0 1" />
+      <limit lower="${shoulder_lift_lower_limit}" upper="${shoulder_lift_upper_limit}"
+        effort="${shoulder_lift_effort_limit}" velocity="${shoulder_lift_velocity_limit}"/>
+      <xacro:if value="${safety_limits}">
+         <safety_controller soft_lower_limit="${shoulder_lift_lower_limit + safety_pos_margin}" soft_upper_limit="${shoulder_lift_upper_limit - safety_pos_margin}" k_position="${safety_k_position}" k_velocity="0.0"/>
+      </xacro:if>
+      <dynamics damping="0" friction="0"/>
+    </joint>
     <joint name="${prefix}elbow_joint" type="revolute">
       <parent link="${prefix}upper_arm_link" />
-      <child link = "${prefix}forearm_link" />
+      <child link="${prefix}forearm_link" />
       <origin xyz="${forearm_x} ${forearm_y} ${forearm_z}" rpy="${forearm_roll} ${forearm_pitch} ${forearm_yaw}" />
-      <axis xyz="0 1 0" />
-      <xacro:unless value="${joint_limited}">
-        <limit lower="${-pi}" upper="${pi}" effort="150.0" velocity="3.15"/>
-      </xacro:unless>
-      <xacro:if value="${joint_limited}">
-        <limit lower="${elbow_joint_lower_limit}" upper="${elbow_joint_upper_limit}" effort="150.0" velocity="3.15"/>
-      </xacro:if>
-      <dynamics damping="0.0" friction="0.0"/>
-    </joint>
-    <link name="${prefix}forearm_link">
-      <visual>
-        <geometry>
-          <mesh filename="package://ur_description/meshes/ur5/visual/forearm.dae" />
-        </geometry>
-        <material name="LightGrey">
-          <color rgba="0.7 0.7 0.7 1.0"/>
-        </material>
-      </visual>
-      <collision>
-        <geometry>
-          <mesh filename="package://ur_description/meshes/ur5/collision/forearm.stl" />
-        </geometry>
-      </collision>
-      <xacro:cylinder_inertial radius="0.06" length="0.5" mass="${forearm_mass}">
-        <origin xyz="0.0 0.0 0.25" rpy="0 0 0" />
-      </xacro:cylinder_inertial>
-    </link>
+      <axis xyz="0 0 1" />
+      <limit lower="${elbow_joint_lower_limit}" upper="${elbow_joint_upper_limit}"
+        effort="${elbow_joint_effort_limit}" velocity="${elbow_joint_velocity_limit}"/>
+      <xacro:if value="${safety_limits}">
+         <safety_controller soft_lower_limit="${elbow_joint_lower_limit + safety_pos_margin}" soft_upper_limit="${elbow_joint_upper_limit - safety_pos_margin}" k_position="${safety_k_position}" k_velocity="0.0"/>
+      </xacro:if>
+      <dynamics damping="0" friction="0"/>
+    </joint>
     <joint name="${prefix}wrist_1_joint" type="revolute">
       <parent link="${prefix}forearm_link" />
-      <child link = "${prefix}wrist_1_link" />
+      <child link="${prefix}wrist_1_link" />
       <origin xyz="${wrist_1_x} ${wrist_1_y} ${wrist_1_z}" rpy="${wrist_1_roll} ${wrist_1_pitch} ${wrist_1_yaw}" />
-      <axis xyz="0 1 0" />
-      <xacro:unless value="${joint_limited}">
-        <limit lower="${-2.0 * pi}" upper="${2.0 * pi}" effort="28.0" velocity="3.2"/>
-      </xacro:unless>
-      <xacro:if value="${joint_limited}">
-        <limit lower="${wrist_1_lower_limit}" upper="${wrist_1_upper_limit}" effort="28.0" velocity="3.2"/>
-      </xacro:if>
-      <dynamics damping="0.0" friction="0.0"/>
-    </joint>
-    <link name="${prefix}wrist_1_link">
-      <visual>
-        <geometry>
-          <mesh filename="package://ur_description/meshes/ur5/visual/wrist1.dae" />
-        </geometry>
-        <material name="LightGrey">
-          <color rgba="0.7 0.7 0.7 1.0"/>
-        </material>
-      </visual>
-      <collision>
-        <geometry>
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
Commit message: Публикатор списка поз

File: src/ur5_husky_main/urdf/robot/trajopt.xacro (robot description, xacro)
@@ -17,5 +17,5 @@
         <origin xyz="0 0 -${wheel_radius - wheel_vertical_offset/2}" rpy="0 0 0" />
         <geometry>
-          <box size="2 2 0.00005"/>
+          <box size="10 10 0.00005"/>
         </geometry>
         <material name="Floor">
@@ -26,11 +26,5 @@
         <origin xyz="0 0 -${wheel_radius - wheel_vertical_offset/2}" rpy="0 0 0" />
         <geometry>
-          <box size="1 1 0.05"/>
-        </geometry>
-      </collision>
-      <collision>
-        <origin xyz="0 0 -${wheel_radius - wheel_vertical_offset/2}" rpy="0 0 0" />
-        <geometry>
-          <box size="1 1 0.05"/>
+          <box size="10 10 0.00005"/>
         </geometry>
       </collision>
