Commit message: Устранено пересечение

File: src/ur5_husky_main/urdf/robot/decorations.urdf.xacro (robot description, xacro)
@@ -11,5 +11,4 @@
     <xacro:property name="husky_front_bumper_extend" value="$(optenv HUSKY_FRONT_BUMPER_EXTEND 0)" />
     <xacro:property name="husky_rear_bumper_extend" value="$(optenv HUSKY_REAR_BUMPER_EXTEND 0)" />
-    <xacro:property name="husky_top_plate" value="$(optenv HUSKY_LARGE_TOP_PLATE true)" />
     <!-- Spawn Husky chassis -->
     <link name="top_chassis_link">
@@ -26,5 +25,5 @@
       <child link="top_chassis_link" />
     </joint>
-    <xacro:if value="$(optenv HUSKY_USER_RAIL_ENABLED true)">
+    <xacro:if value="$(optenv HUSKY_USER_RAIL_ENABLED false)">
       <!-- Spawn user rails -->
       <link name="user_rail_link">
@@ -119,5 +118,5 @@
           <parent link="base_link" />
           <child link="top_plate_link"/>
-          <origin xyz="0.0812 0 0.225" rpy="0 0 0"/>
+          <origin xyz="0.0812 0 0.2255" rpy="0 0 0"/>
         </joint>
         <!-- Top plate front link -->

Commit message: Модель робота

File: src/ur5_husky_main/urdf/robot/decorations.urdf.xacro (robot description, xacro)
@@ -97,7 +97,7 @@
       </joint>
     </xacro:if>
-    <xacro:if value="$(optenv HUSKY_TOP_PLATE_ENABLED true)">
+    <!-- <xacro:if value="$(optenv HUSKY_TOP_PLATE_ENABLED true)"> -->
       <!-- Spawn the top plate -->
-      <xacro:if value="$(optenv HUSKY_LARGE_TOP_PLATE true)">
+      <!-- <xacro:if value="$(optenv HUSKY_LARGE_TOP_PLATE true)"> -->
         <link name="top_plate_link">
           <visual>
@@ -132,6 +132,6 @@
           <origin xyz="-0.4125 0 0.00672" rpy="0 0 0"/>
         </joint>
-      </xacro:if>
-      <xacro:unless value="$(optenv HUSKY_LARGE_TOP_PLATE true)">
+      <!-- </xacro:if> -->
+      <!-- <xacro:unless value="$(optenv HUSKY_LARGE_TOP_PLATE true)">
         <link name="top_plate_link">
           <visual>
@@ -147,27 +147,27 @@
             </geometry>
           </collision>
-        </link>
+        </link>-->
         <!-- Attach top plate -->
-        <joint name="top_plate_joint" type="fixed">
+        <!-- <joint name="top_plate_joint" type="fixed">
           <parent link="base_link" />
           <child link="top_plate_link"/>
           <origin xyz="0.0812 0 0.245" rpy="0 0 0"/>
-        </joint>
+        </joint> -->
         <!-- Top plate front link -->
-        <joint name="top_plate_front_joint" type="fixed">
+        <!-- <joint name="top_plate_front_joint" type="fixed">
           <parent link="top_plate_link" />
           <child link="top_plate_front_link"/>
           <origin xyz="0.36367 0 0.00639" rpy="0 0 0"/>
-        </joint>
+        </joint> -->
         <!-- Top plate rear link-->
-        <joint name="top_plate_rear_joint" type="fixed">
+        <!--<joint name="top_plate_rear_joint" type="fixed">
           <parent link="top_plate_link" />
           <child link="top_plate_rear_link"/>
           <origin xyz="-0.36633 0 0.00639" rpy="0 0 0"/>
         </joint>
-      </xacro:unless>
+      </xacro:unless> -->
       <link name="top_plate_front_link"/>
       <link name="top_plate_rear_link"/>
-    </xacro:if>
+    <!-- </xacro:if> -->
   </xacro:macro>
 </robot>

File: src/ur5_husky_main/urdf/robot/husky.xacro (robot description, xacro)
@@ -55,5 +55,5 @@
         </geometry>
       </visual>
-      <collision>
+      <!-- <collision>
         <origin xyz="${( husky_front_bumper_extend - husky_rear_bumper_extend ) / 2.0} 0 ${base_z_size/4}" rpy="0 0 0" />
         <geometry>
@@ -66,5 +66,5 @@
           <box size="${base_x_size*4/5} ${base_y_size} ${base_z_size/2-0.02}"/>
         </geometry>
-      </collision>
+      </collision> -->
     </link>
     <!-- Base footprint is on the ground under the robot -->
@@ -108,10 +108,10 @@
           <inertia ixx="0.00000001" ixy="0.00000001" ixz="0.00000001" iyy="0.00000001" iyz="0.00000001" izz="0.00000001"/>
       </inertial>
-      <collision name="base_link_fixed_joint_lump__robot/bumper_link">
+      <!-- <collision name="base_link_fixed_joint_lump__robot/bumper_link">
           <origin rpy="0 0 0" xyz="0 0 0.1"/>
           <geometry>
               <box size="1.0 0.7 0.31"/>
           </geometry>
-      </collision>
+      </collision> -->
     </link>
     <joint name="bumper_joint" type="fixed">
